Commit message: mejora de paso

File: ros2/install/march_description/share/march_description/urdf/marchS.xacro (robot description, xacro)
@@ -334,7 +334,7 @@
         </inertial>
         <collision>
-            <origin xyz="0 ${lower_leg_width_y + 0.01} 0" rpy="0 0 0"/>
-            <geometry>
-                <box size="0.17 0.13 0.12"/>
+            <origin xyz="0 ${-lower_leg_width_y/2 - 0.055} -0.05" rpy="0 0 0"/>
+            <geometry>
+                <box size="0.17 0.15 0.10"/>
             </geometry>
         </collision>
@@ -520,7 +520,7 @@
         </inertial>
         <collision>
-            <origin xyz="0 ${-lower_leg_width_y/2 -0.03} 0" rpy="0 0 0"/>
-            <geometry>
-                <box size="0.17 0.13 0.12"/>
+            <origin xyz="0 ${-lower_leg_width_y/2 - 0.055} -0.05" rpy="0 0 0"/>
+            <geometry>
+                <box size="0.17 0.15 0.10"/>
             </geometry>
         </collision>
